File: PCB/Pico_Handheld/Pico_Handheld.kicad_pcb (KiCad board)
At the start: 2 copper layers, 86.4 x 91.4 mm, 15 parts, among them SW1 UP, SW2 SW_SPDT, SW3 DOWN, SW4 LEFT, SW5 RIGHT, SW6 B, SW7 A, U1 Pico, U2 Volume_Wheel, U3 128x64_OLED

Commit message: V0.1.1 Finalised PCB V1.0
Parts:
- BZ1: footprint Buzzer_Beeper:Buzzer_12x9.5RM7.6 -> Buzzer_Beeper:MagneticBuzzer_ProSignal_ABT-410-RC
- U3: value 128x64_OLED -> 0.91_128x64_SSD1306_Oled_Display
Other:
- board text added: "Pico Handheld Games Console"
- board text added: "Sean Price"
- board text added: "V1.0"
Changed lines of the file:
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@@
       (layerselection 0x00010fc_ffffffff)
       (disableapertmacros false)
-      (usegerberextensions false)
-      (usegerberattributes true)
-      (usegerberadvancedattributes true)
-      (creategerberjobfile true)
+      (usegerberextensions true)
+      (usegerberattributes false)
+      (usegerberadvancedattributes false)
+      (creategerberjobfile false)
       (svguseinch false)
       (svgprecision 6)
@@
       (plotinvisibletext false)
       (sketchpadsonfab false)
-      (subtractmaskfromsilk false)
+      (subtractmaskfromsilk true)
       (outputformat 1)
       (mirror false)
-      (drillshape 1)
+      (drillshape 0)
       (scaleselection 1)
-      (outputdirectory "")
+      (outputdirectory "../Pico_Handheld_V1_Gerber/")
     )
   )
@@
       (net 12 "GPIO10") (pinfunction "2") (pintype "passive"))
   )
-  (footprint "Buzzer_Beeper:Buzzer_12x9.5RM7.6" (layer "F.Cu")
+  (footprint "Buzzer_Beeper:MagneticBuzzer_ProSignal_ABT-410-RC" (layer "F.Cu")
     (at 171.46 66.04)
-    (descr "Generic Buzzer, D12mm height 9.5mm with RM7.6mm")
-    (tags "buzzer")
+    (descr "Buzzer, Elektromagnetic Beeper, Summer, 1,5V-DC,")
+    (tags "Pro Signal ABT-410-RC ")
     (property "Sheetfile" "Pico_Handheld.kicad_sch")
     (property "Sheetname" "")
     (attr through_hole)
-    (fp_text reference "BZ1" (at 3.8 -7.2) (layer "F.SilkS")
-      (effects (font (size 1 1) (thickness 0.15)))
-    )
-    (fp_text value "Buzzer" (at 3.8 7.4) (layer "F.Fab")
-      (effects (font (size 1 1) (thickness 0.15)))
-    )
-    (fp_text user "+" (at -0.01 -2.54) (layer "F.SilkS")
-      (effects (font (size 1 1) (thickness 0.15)))
-    )
-    (fp_text user "+" (at -0.01 -2.54) (layer "F.Fab")
-      (effects (font (size 1 1) (thickness 0.15)))
-    )
-    (fp_text user "${REFERENCE}" (at 3.8 -4) (layer "F.Fab")
-      (effects (font (size 1 1) (thickness 0.15)))
-    )
-    (fp_circle (center 3.8 0) (end 9.9 0) (layer "F.SilkS") (width 0.12) (fill none))
-    (fp_circle (center 3.8 0) (end 10.05 0) (layer "F.CrtYd") (width 0.05) (fill none))
-    (fp_circle (center 3.8 0) (end 4.8 0) (layer "F.Fab") (width 0.1) (fill none))
-    (fp_circle (center 3.8 0) (end 9.8 0) (layer "F.Fab") (width 0.1) (fill none))
-    (pad "1" thru_hole rect (at 0 0) (size 2 2) (drill 1) (layers *.Cu *.Mask)
+    (fp_text reference "BZ1" (at 3.25 -7) (layer "F.SilkS")
+      (effects (font (size 1 1) (thickness 0.15)))
+    )
+    (fp_text value "Buzzer" (at 3.25 7) (layer "F.Fab")
+      (effects (font (size 1 1) (thickness 0.15)))
+    )
+    (fp_text user "+" (at 0 -1.8) (layer "F.SilkS")
+      (effects (font (size 1 1) (thickness 0.15)))
+    )
+    (fp_text user "+" (at 0 -1.8) (layer "F.Fab")
+      (effects (font (size 1 1) (thickness 0.15)))
+    )
+    (fp_text user "${REFERENCE}" (at 3.25 -7) (layer "F.Fab")
+      (effects (font (size 1 1) (thickness 0.15)))
+    )
+    (fp_circle (center 3.25 0) (end 9.35 0) (layer "F.SilkS") (width 0.12) (fill none))
+    (fp_circle (center 3.25 0) (end 9.5 0) (layer "F.CrtYd") (width 0.05) (fill none))
+    (fp_circle (center 3.25 0) (end 4.4 0) (layer "F.Fab") (width 0.1) (fill none))
+    (fp_circle (center 3.25 0) (end 9.25 0) (layer "F.Fab") (width 0.1) (fill none))
+    (pad "1" thru_hole rect (at 0 0) (size 1.6 1.6) (drill 1) (layers *.Cu *.Mask)
       (net 3 "Net-(BZ1-Pad1)") (pinfunction "-") (pintype "passive"))
-    (pad "2" thru_hole circle (at 7.6 0) (size 2 2) (drill 1) (layers *.Cu *.Mask)
+    (pad "2" thru_hole circle (at 6.5 0) (size 1.6 1.6) (drill 1) (layers *.Cu *.Mask)
       (net 2 "GND") (pinfunction "+") (pintype "passive"))
-    (model "${KICAD6_3DMODEL_DIR}/Buzzer_Beeper.3dshapes/Buzzer_12x9.5RM7.6.wrl"
+    (model "${KICAD6_3DMODEL_DIR}/Buzzer_Beeper.3dshapes/MagneticBuzzer_ProSignal_ABT-410-RC.wrl"
       (offset (xyz 0 0 0))
       (scale (xyz 1 1 1))
@@
       (effects (font (size 1 1) (thickness 0.15)))
     )
+    (fp_line (start -7.112 5.08) (end 1.524 5.08) (layer "F.SilkS") (width 0.12))
+    (fp_line (start -7.62 -3.048) (end -7.62 -1.016) (layer "F.SilkS") (width 0.12))
+    (fp_line (start -7.62 1.016) (end -7.62 3.048) (layer "F.SilkS") (width 0.12))
     (fp_line (start -7.112 -5.08) (end 1.524 -5.08) (layer "F.SilkS") (width 0.12))
-    (fp_line (start -7.62 1.016) (end -7.62 3.048) (layer "F.SilkS") (width 0.12))
-    (fp_line (start -7.62 -3.048) (end -7.62 -1.016) (layer "F.SilkS") (width 0.12))
-    (fp_line (start -7.112 5.08) (end 1.524 5.08) (layer "F.SilkS") (width 0.12))
     (fp_arc (start 3.556 -5.08) (mid 6.20093 0) (end 3.556 5.08) (layer "F.SilkS") (width 0.12))
     (fp_circle (center 0 0) (end -8.636 0) (layer "F.SilkS") (width 0.12) (fill none))
@@
     (pad "3" thru_hole circle (at -7.62 4.064) (size 1.524 1.524) (drill 0.762) (layers *.Cu *.Mask)
       (net 2 "GND") (pintype "passive"))
-    (pad "4" thru_hole circle (at 2.54 -5.08) (size 1.524 1.524) (drill 0.762) (layers *.Cu *.Mask)
+    (pad "4" thru_hole circle (at 2.54 -5.08) (size 2 2) (drill 1) (layers *.Cu *.Mask)
       (net 17 "unconnected-(U2-Pad4)") (pintype "passive+no_connect"))
-    (pad "5" thru_hole circle (at 2.54 5.08) (size 1.524 1.524) (drill 0.762) (layers *.Cu *.Mask)
+    (pad "5" thru_hole circle (at 2.54 5.08) (size 2 2) (drill 1) (layers *.Cu *.Mask)
       (net 18 "unconnected-(U2-Pad5)") (pintype "passive+no_connect"))
   )
@@
       (effects (font (size 1 1) (thickness 0.15)))
     )
-    (fp_text value "128x64_OLED" (at 0 -10.67 unlocked) (layer "F.Fab")
+    (fp_text value "0.91_128x64_SSD1306_Oled_Display" (at 0 -10.67 unlocked) (layer "F.Fab")
       (effects (font (size 1 1) (thickness 0.15)))
     )
@@
   (gr_line (start 153.67 49.53) (end 110.49 49.53) (layer "Edge.Cuts") (width 0.1))
   (gr_line (start 196.85 49.53) (end 196.85 140.97) (layer "Edge.Cuts") (width 0.1))
+  (gr_text "Pico Handheld Games Console" (at 158.75 93.345) (layer "F.SilkS")
+    (effects (font (size 1 1) (thickness 0.15)) (justify left))
+  )
+  (gr_text "V1.0" (at 158.75 95.25) (layer "F.SilkS")
+    (effects (font (size 1 1) (thickness 0.15)) (justify left))
+  )
   (gr_text "Vcc/GND/SCL/SDA" (at 153.67 65.405) (layer "F.SilkS")
     (effects (font (size 1 1) (thickness 0.15)))
@@
     (effects (font (size 1 1) (thickness 0.15)))
   )
+  (gr_text "Sean Price" (at 158.75 97.155) (layer "F.SilkS")
+    (effects (font (size 1 1) (thickness 0.15)) (justify left))
+  )
   (segment (start 185.42 52.07) (end 185.42 53.975) (width 1.5) (layer "B.Cu") (net 1))
